File: dac-brd/dac-brd.kicad_pcb (KiCad board)
At the start: 2 copper layers, 51 x 53 mm, 18 parts, among them J1 HTR, J3 UART, U1 REF5030ID, U2 DAC5578xPW, U3 DAC5578xPW

Commit message: Finished mezzanine layout
Parts:
- added J2: I2C, Connector_PinHeader_2.54mm:PinHeader_1x04_P2.54mm_Vertical, F.Cu at (136.5, 102.5)
- moved J3 14.0 mm to (136.5, 88.0)
Connections:
- A1 pad 22: unconnected-(A1-GPIO17-Pad22)_1 -> /LED_PWM
- A1 pad 4: /LED_PWM -> /SDA1
- A1 pad 5: unconnected-(A1-GPIO3-Pad5) -> /SCL1
Routing:
- net /LED_PWM: track 63.2 -> 21.0 mm
- net /SDA1: track 0.00 -> 22.9 mm
- net +3V3: track 7.37 -> 28.0 mm
- net /SCL1: track 0.00 -> 17.5 mm
- net /RX: track 25.0 -> 9.86 mm
- net /TX: track 24.5 -> 9.65 mm
- net GND: vias 144 -> 156
Other:
- board text added: "3V3 SCL SDA GND"
